File: rpi.sch (KiCad schematic (older format))
At the start: 18 parts, among them J1 M20-7832046, Q1 DMMT5401, Q2 DMG2305UX, U1 CAT24C32

Commit message: Added manufacturer number to schematic
Parts:
- C1: manf# (none) -> C0603C104M5RACTU
- J1: manf# (none) -> M20-7832046
- JP1: manf# (none) -> M20-9990246
- Q1: manf# (none) -> DMMT5401
- Q2: manf# (none) -> DMG2305UX
- R1, R5: manf# (none) -> CR0603-FX-4702ELF
- R2, R3: manf# (none) -> RC0603FR-103K9L
- R4: manf# (none) -> AC0603FR-0710KL
- U1: manf# (none) -> CAT24C32WI-GT3
Changed lines of the file:
@@
 F 2 "Connector_PinSocket_2.54mm:PinSocket_2x20_P2.54mm_Vertical" H 3250 1300 50  0001 C CNN
 F 3 "https://eu.mouser.com/datasheet/2/181/M20-783-1133465.pdf" H 2550 1100 50  0000 C CNN
+F 4 "M20-7832046" H 0   0   50  0001 C CNN "manf#"
 	1    3250 1100
 	1    0    0    -1
@@
 F 2 "Package_TO_SOT_SMD:SOT-23" H 8000 1450 50  0001 C CNN
 F 3 "https://www.diodes.com/assets/Datasheets/DMG2305UX.pdf" H 7800 1350 50  0001 C CNN
+F 4 "DMG2305UX" H 0   0   50  0001 C CNN "manf#"
 	1    7800 1350
 	0    -1   -1   0
@@
 F 2 "Resistor_SMD:R_0603_1608Metric" V 8130 2450 50  0001 C CNN
 F 3 "" H 8200 2450 50  0001 C CNN
+F 4 "CR0603-FX-4702ELF" H 0   0   50  0001 C CNN "manf#"
 	1    8200 2450
 	1    0    0    -1
@@
 F 2 "Package_SO:SOIC-8_3.9x4.9mm_P1.27mm" H 2850 5000 50  0001 C CNN
 F 3 "" H 2850 5000 50  0000 C CNN
+F 4 "CAT24C32WI-GT3" H 0   0   50  0001 C CNN "manf#"
 	1    2850 5000
 	1    0    0    -1
@@
 F 2 "Resistor_SMD:R_0603_1608Metric" V 3980 4650 50  0001 C CNN
 F 3 "" H 4050 4650 50  0001 C CNN
+F 4 "RC0603FR-103K9L" H 0   0   50  0001 C CNN "manf#"
 	1    4050 4650
 	0    1    1    0
@@
 F 2 "Resistor_SMD:R_0603_1608Metric" V 3980 4800 50  0001 C CNN
 F 3 "" H 4050 4800 50  0001 C CNN
+F 4 "RC0603FR-103K9L" H 0   0   50  0001 C CNN "manf#"
 	1    4050 4800
 	0    1    1    0
@@
 F 2 "Package_TO_SOT_SMD:SOT-23-6" H 7691 1941 50  0001 L CIN
 F 3 "" H 7500 1850 50  0000 L CNN
+F 4 "DMMT5401" H 0   0   50  0001 C CNN "manf#"
 	1    7500 1850
 	-1   0    0    1
@@
 F 2 "Package_TO_SOT_SMD:SOT-23-6" H 8291 1941 50  0001 L CIN
 F 3 "" H 8100 1850 50  0000 L CNN
+F 4 "DMMT5401" H 0   0   50  0001 C CNN "manf#"
 	2    8100 1850
 	1    0    0    1
@@
 F 2 "Connector_PinHeader_2.54mm:PinHeader_1x02_P2.54mm_Vertical" H 1850 5200 50  0001 C CNN
 F 3 "~" H 1850 5200 50  0001 C CNN
+F 4 "M20-9990246" H 0   0   50  0001 C CNN "manf#"
 	1    1850 5200
 	1    0    0    -1
@@
 F 2 "Resistor_SMD:R_0603_1608Metric" V 1830 5400 50  0001 C CNN
 F 3 "" H 1900 5400 50  0001 C CNN
+F 4 "CR0603-FX-4702ELF" H 0   0   50  0001 C CNN "manf#"
 	1    1900 5400
 	0    1    1    0
@@
 F 2 "Resistor_SMD:R_0603_1608Metric" V 7330 2450 50  0001 C CNN
 F 3 "" H 7400 2450 50  0001 C CNN
+F 4 "AC0603FR-0710KL" H 0   0   50  0001 C CNN "manf#"
 	1    7400 2450
 	1    0    0    -1
@@
 F 2 "Capacitor_SMD:C_0603_1608Metric" H 3438 4450 50  0001 C CNN
 F 3 "~" H 3400 4600 50  0001 C CNN
+F 4 "C0603C104M5RACTU" H 0   0   50  0001 C CNN "manf#"
 	1    3400 4600
 	1    0    0    -1
