File: connectors.sch (KiCad schematic (older format))
At the start: 43 parts, among them J12 20021121-00010C4LF, J13 70543-0001, J14 70543-0001, J15 70543-0001, J16 70543-0001, J17 70543-0001, J18 70543-0001, J19 70543-0001, J20 70543-0001, J21 70543-0003, J22 70543-0002, J23 70543-0002, J24 70543-0002, J25 Conn_02x20_Odd_Even

Commit message: Added manufacturer number to schematic
Parts:
- C112, C113, C114, C115: manf# (none) -> C0603C104M5RACTU
- D14, D15, D16, D17, D18, D19, D20, D21, D22, D23, D24, D25, D26, D27: manf# (none) -> BAT54GWJ
- J12: manf# (none) -> 20021121-00010C4LF
- J13, J14, J15, J16, J17, J18, J19, J20: manf# (none) -> 70543-0001
- J21: manf# (none) -> 70543-0003
- J22, J23, J24: manf# (none) -> 70543-0002
- J25: manf# (none) -> 95157-140LF
- R119, R120, R121, R122, R123, R124, R125, R126: manf# (none) -> AC0603JR-074K7L
- R127, R128, R129: manf# (none) -> RC0603JR-7W1KL
Changed lines of the file:
@@
 F 2 "Resistor_SMD:R_0603_1608Metric" V 2080 3300 50  0001 C CNN
 F 3 "~" H 2150 3300 50  0001 C CNN
+F 4 "AC0603JR-074K7L" H 0   0   50  0001 C CNN "manf#"
 	1    2150 3300
 	0    1    1    0
@@
 F 2 "Resistor_SMD:R_0603_1608Metric" V 2430 3050 50  0001 C CNN
 F 3 "~" H 2500 3050 50  0001 C CNN
+F 4 "AC0603JR-074K7L" H 0   0   50  0001 C CNN "manf#"
 	1    2500 3050
 	1    0    0    -1
@@
 F 2 "heteromycin:70543-0001" H 2800 3300 50  0001 C CNN
 F 3 "" H 2800 3300 50  0001 C CNN
+F 4 "70543-0001" H 0   0   50  0001 C CNN "manf#"
 	1    2800 3300
 	1    0    0    -1
@@
 F 2 "Capacitor_SMD:C_0603_1608Metric" H 1088 3300 50  0001 C CNN
 F 3 "~" H 1050 3450 50  0001 C CNN
+F 4 "C0603C104M5RACTU" H 0   0   50  0001 C CNN "manf#"
 	1    1050 3450
 	1    0    0    -1
@@
 F 2 "Connector_PinHeader_1.27mm:PinHeader_2x05_P1.27mm_Vertical_SMD" H 1500 1650 50  0001 C CNN
 F 3 "https://www.mouser.de/datasheet/2/18/20021121-1362884.pdf" H 1500 1650 50  0001 C CNN
+F 4 "20021121-00010C4LF" H 0   0   50  0001 C CNN "manf#"
 	1    1500 1650
 	1    0    0    -1
@@
 F 2 "heteromycin:70543-0003" H 4800 3100 50  0001 C CNN
 F 3 "https://www.mouser.de/ProductDetail/Molex/70543-0003?qs=sGAEpiMZZMs%252bGHln7q6pm%252bS0pk2Wo0XxCD3CKlCQrmU%3d" H 4800 3100 50  0001 C CNN
+F 4 "70543-0003" H 0   0   50  0001 C CNN "manf#"
 	1    4800 3100
 	1    0    0    -1
@@
 F 2 "Resistor_SMD:R_0603_1608Metric" V 4980 4500 50  0001 C CNN
 F 3 "~" H 5050 4500 50  0001 C CNN
+F 4 "RC0603JR-7W1KL" H 0   0   50  0001 C CNN "manf#"
 	1    5050 4500
 	0    1    1    0
@@
 F 2 "Resistor_SMD:R_0603_1608Metric" V 4980 5700 50  0001 C CNN
 F 3 "~" H 5050 5700 50  0001 C CNN
+F 4 "RC0603JR-7W1KL" H 0   0   50  0001 C CNN "manf#"
 	1    5050 5700
 	0    1    1    0
@@
 F 2 "Resistor_SMD:R_0603_1608Metric" V 4980 6900 50  0001 C CNN
 F 3 "~" H 5050 6900 50  0001 C CNN
+F 4 "RC0603JR-7W1KL" H 0   0   50  0001 C CNN "manf#"
 	1    5050 6900
 	0    1    1    0
@@
 F 2 "Resistor_SMD:R_0603_1608Metric" V 2080 4500 50  0001 C CNN
 F 3 "~" H 2150 4500 50  0001 C CNN
+F 4 "AC0603JR-074K7L" H 0   0   50  0001 C CNN "manf#"
 	1    2150 4500
 	0    1    1    0
@@
 F 2 "Resistor_SMD:R_0603_1608Metric" V 2430 4250 50  0001 C CNN
 F 3 "~" H 2500 4250 50  0001 C CNN
+F 4 "AC0603JR-074K7L" H 0   0   50  0001 C CNN "manf#"
 	1    2500 4250
 	1    0    0    -1
@@
 F 2 "Capacitor_SMD:C_0603_1608Metric" H 1088 4500 50  0001 C CNN
 F 3 "~" H 1050 4650 50  0001 C CNN
+F 4 "C0603C104M5RACTU" H 0   0   50  0001 C CNN "manf#"
 	1    1050 4650
 	1    0    0    -1
@@
 F 2 "Resistor_SMD:R_0603_1608Metric" V 2080 5700 50  0001 C CNN
 F 3 "~" H 2150 5700 50  0001 C CNN
+F 4 "AC0603JR-074K7L" H 0   0   50  0001 C CNN "manf#"
 	1    2150 5700
 	0    1    1    0
@@
 F 2 "Resistor_SMD:R_0603_1608Metric" V 2430 5450 50  0001 C CNN
 F 3 "~" H 2500 5450 50  0001 C CNN
+F 4 "AC0603JR-074K7L" H 0   0   50  0001 C CNN "manf#"
 	1    2500 5450
 	1    0    0    -1
@@
 F 2 "Capacitor_SMD:C_0603_1608Metric" H 1088 5700 50  0001 C CNN
 F 3 "~" H 1050 5850 50  0001 C CNN
+F 4 "C0603C104M5RACTU" H 0   0   50  0001 C CNN "manf#"
 	1    1050 5850
 	1    0    0    -1
@@
 F 2 "Resistor_SMD:R_0603_1608Metric" V 2080 6900 50  0001 C CNN
 F 3 "~" H 2150 6900 50  0001 C CNN
+F 4 "AC0603JR-074K7L" H 0   0   50  0001 C CNN "manf#"
 	1    2150 6900
 	0    1    1    0
@@
 F 2 "Resistor_SMD:R_0603_1608Metric" V 2430 6650 50  0001 C CNN
 F 3 "~" H 2500 6650 50  0001 C CNN
+F 4 "AC0603JR-074K7L" H 0   0   50  0001 C CNN "manf#"
 	1    2500 6650
 	1    0    0    -1
@@
 F 2 "Capacitor_SMD:C_0603_1608Metric" H 1088 6900 50  0001 C CNN
 F 3 "~" H 1050 7050 50  0001 C CNN
+F 4 "C0603C104M5RACTU" H 0   0   50  0001 C CNN "manf#"
 	1    1050 7050
 	1    0    0    -1
@@
 F 2 "heteromycin:70543-0001" H 4800 1300 50  0001 C CNN
 F 3 "https://www.mouser.de/ProductDetail/Molex/50-57-9402?qs=%2fha2pyFadujDsSJKPzBRyOySofHgnbNURyOy7MwFkp4%3d" H 4800 1300 50  0001 C CNN
+F 4 "70543-0001" H 0   0   50  0001 C CNN "manf#"
 	1    4800 1300
 	1    0    0    -1
@@
 F 2 "Connector_PinHeader_2.54mm:PinHeader_2x20_P2.54mm_Vertical_SMD" H 8350 2200 50  0001 C CNN
 F 3 "~" H 8350 2200 50  0001 C CNN
+F 4 "95157-140LF" H 0   0   50  0001 C CNN "manf#"
 	1    8350 2200
 	1    0    0    -1
@@
 F 2 "heteromycin:70543-0001" H 4800 1600 50  0001 C CNN
 F 3 "https://www.mouser.de/ProductDetail/Molex/50-57-9402?qs=%2fha2pyFadujDsSJKPzBRyOySofHgnbNURyOy7MwFkp4%3d" H 4800 1600 50  0001 C CNN
+F 4 "70543-0001" H 0   0   50  0001 C CNN "manf#"
 	1    4800 1600
 	1    0    0    -1
@@
 F 2 "heteromycin:70543-0001" H 4800 1900 50  0001 C CNN
 F 3 "https://www.mouser.de/ProductDetail/Molex/50-57-9402?qs=%2fha2pyFadujDsSJKPzBRyOySofHgnbNURyOy7MwFkp4%3d" H 4800 1900 50  0001 C CNN
+F 4 "70543-0001" H 0   0   50  0001 C CNN "manf#"
 	1    4800 1900
 	1    0    0    -1
@@
 F 2 "heteromycin:70543-0001" H 4800 2200 50  0001 C CNN
 F 3 "https://www.mouser.de/ProductDetail/Molex/50-57-9402?qs=%2fha2pyFadujDsSJKPzBRyOySofHgnbNURyOy7MwFkp4%3d" H 4800 2200 50  0001 C CNN
+F 4 "70543-0001" H 0   0   50  0001 C CNN "manf#"
 	1    4800 2200
 	1    0    0    -1
@@
 F 2 "heteromycin:70543-0001" H 2800 4500 50  0001 C CNN
 F 3 "" H 2800 4500 50  0001 C CNN
+F 4 "70543-0001" H 0   0   50  0001 C CNN "manf#"
 	1    2800 4500
 	1    0    0    -1
@@
 F 2 "heteromycin:70543-0001" H 2800 5700 50  0001 C CNN
 F 3 "" H 2800 5700 50  0001 C CNN
+F 4 "70543-0001" H 0   0   50  0001 C CNN "manf#"
 	1    2800 5700
 	1    0    0    -1
@@
 F 2 "heteromycin:70543-0001" H 2800 6900 50  0001 C CNN
 F 3 "" H 2800 6900 50  0001 C CNN
+F 4 "70543-0001" H 0   0   50  0001 C CNN "manf#"
 	1    2800 6900
 	1    0    0    -1
@@
 F 2 "heteromycin:70543-0002" H 5750 4600 50  0001 C CNN
 F 3 "~" H 5750 4600 50  0001 C CNN
+F 4 "70543-0002" H 0   0   50  0001 C CNN "manf#"
 	1    5750 4600
 	1    0    0    -1
@@
 F 2 "heteromycin:70543-0002" H 5750 5800 50  0001 C CNN
 F 3 "~" H 5750 5800 50  0001 C CNN
+F 4 "70543-0002" H 0   0   50  0001 C CNN "manf#"
 	1    5750 5800
 	1    0    0    -1
@@
 F 2 "heteromycin:70543-0002" H 5750 7000 50  0001 C CNN
 F 3 "~" H 5750 7000 50  0001 C CNN
+F 4 "70543-0002" H 0   0   50  0001 C CNN "manf#"
 	1    5750 7000
 	1    0    0    -1
@@
 F 2 "Diode_SMD:D_SOD-123" H 1500 3050 50  0001 C CNN
 F 3 "https://www.mouser.de/datasheet/2/916/BAT54GW-1318921.pdf" H 1500 3050 50  0001 C CNN
+F 4 "BAT54GWJ" H 0   0   50  0001 C CNN "manf#"
 	1    1500 3050
 	0    1    1    0
@@
 F 2 "Diode_SMD:D_SOD-123" H 1500 4250 50  0001 C CNN
 F 3 "https://www.mouser.de/datasheet/2/916/BAT54GW-1318921.pdf" H 1500 4250 50  0001 C CNN
+F 4 "BAT54GWJ" H 0   0   50  0001 C CNN "manf#"
 	1    1500 4250
 	0    1    1    0
@@
 F 2 "Diode_SMD:D_SOD-123" H 1500 4750 50  0001 C CNN
 F 3 "https://www.mouser.de/datasheet/2/916/BAT54GW-1318921.pdf" H 1500 4750 50  0001 C CNN
+F 4 "BAT54GWJ" H 0   0   50  0001 C CNN "manf#"
 	1    1500 4750
 	0    1    1    0
@@
 F 2 "Diode_SMD:D_SOD-123" H 1500 5450 50  0001 C CNN
 F 3 "https://www.mouser.de/datasheet/2/916/BAT54GW-1318921.pdf" H 1500 5450 50  0001 C CNN
+F 4 "BAT54GWJ" H 0   0   50  0001 C CNN "manf#"
 	1    1500 5450
 	0    1    1    0
@@
 F 2 "Diode_SMD:D_SOD-123" H 1500 5950 50  0001 C CNN
 F 3 "https://www.mouser.de/datasheet/2/916/BAT54GW-1318921.pdf" H 1500 5950 50  0001 C CNN
+F 4 "BAT54GWJ" H 0   0   50  0001 C CNN "manf#"
 	1    1500 5950
 	0    1    1    0
@@
 F 2 "Diode_SMD:D_SOD-123" H 1500 6650 50  0001 C CNN
 F 3 "https://www.mouser.de/datasheet/2/916/BAT54GW-1318921.pdf" H 1500 6650 50  0001 C CNN
+F 4 "BAT54GWJ" H 0   0   50  0001 C CNN "manf#"
 	1    1500 6650
 	0    1    1    0
@@
 F 2 "Diode_SMD:D_SOD-123" H 1500 7150 50  0001 C CNN
 F 3 "https://www.mouser.de/datasheet/2/916/BAT54GW-1318921.pdf" H 1500 7150 50  0001 C CNN
+F 4 "BAT54GWJ" H 0   0   50  0001 C CNN "manf#"
 	1    1500 7150
 	0    1    1    0
@@
 F 2 "Diode_SMD:D_SOD-123" H 4500 7150 50  0001 C CNN
 F 3 "https://www.mouser.de/datasheet/2/916/BAT54GW-1318921.pdf" H 4500 7150 50  0001 C CNN
+F 4 "BAT54GWJ" H 0   0   50  0001 C CNN "manf#"
 	1    4500 7150
 	0    1    1    0
@@
 F 2 "Diode_SMD:D_SOD-123" H 4500 6650 50  0001 C CNN
 F 3 "https://www.mouser.de/datasheet/2/916/BAT54GW-1318921.pdf" H 4500 6650 50  0001 C CNN
+F 4 "BAT54GWJ" H 0   0   50  0001 C CNN "manf#"
 	1    4500 6650
 	0    1    1    0
@@
 F 2 "Diode_SMD:D_SOD-123" H 4500 5950 50  0001 C CNN
 F 3 "https://www.mouser.de/datasheet/2/916/BAT54GW-1318921.pdf" H 4500 5950 50  0001 C CNN
+F 4 "BAT54GWJ" H 0   0   50  0001 C CNN "manf#"
 	1    4500 5950
 	0    1    1    0
@@
 F 2 "Diode_SMD:D_SOD-123" H 4500 4750 50  0001 C CNN
 F 3 "https://www.mouser.de/datasheet/2/916/BAT54GW-1318921.pdf" H 4500 4750 50  0001 C CNN
+F 4 "BAT54GWJ" H 0   0   50  0001 C CNN "manf#"
 	1    4500 4750
 	0    1    1    0
@@
 F 2 "Diode_SMD:D_SOD-123" H 4500 4250 50  0001 C CNN
 F 3 "https://www.mouser.de/datasheet/2/916/BAT54GW-1318921.pdf" H 4500 4250 50  0001 C CNN
+F 4 "BAT54GWJ" H 0   0   50  0001 C CNN "manf#"
 	1    4500 4250
 	0    1    1    0
@@
 F 2 "Diode_SMD:D_SOD-123" H 4500 5450 50  0001 C CNN
 F 3 "https://www.mouser.de/datasheet/2/916/BAT54GW-1318921.pdf" H 4500 5450 50  0001 C CNN
+F 4 "BAT54GWJ" H 0   0   50  0001 C CNN "manf#"
 	1    4500 5450
 	0    1    1    0
@@
 F 2 "Diode_SMD:D_SOD-123" H 1500 3550 50  0001 C CNN
 F 3 "https://www.mouser.de/datasheet/2/916/BAT54GW-1318921.pdf" H 1500 3550 50  0001 C CNN
+F 4 "BAT54GWJ" H 0   0   50  0001 C CNN "manf#"
 	1    1500 3550
 	0    1    1    0
