File: mosfets.sch (KiCad schematic (older format))
At the start: 28 parts, among them Q11 PSMN1R2-30YLC,115, Q12 PSMN1R2-30YLC,115, Q13 PSMN1R2-30YLC,115, Q14 IRLML0030TRPbF, Q15 IRLML0030TRPbF, Q16 IRLML0030TRPbF, Q17 IRLML0030TRPbF

Commit message: Added manufacturer number to schematic
Parts:
- D10, D11, D12, D13: manf# (none) -> BAT54GWJ
- D7, D8, D9: manf# (none) -> SK310A-LTP
- Q11, Q12, Q13: manf# (none) -> PSMN1R2-30YLC,115
- Q14, Q15, Q16, Q17: manf# (none) -> IRLML0030TRPbF
- R31, R32, R33, R37, R38, R41, R42: manf# (none) -> RC0603FR-7W100RL
- R34, R35, R36, R39, R40, R43, R44: manf# (none) -> CRCW0603100KFKEAC
Changed lines of the file:
@@
 F 2 "Diode_SMD:D_SMA" H 2000 1300 50  0001 C CNN
 F 3 "https://www.mouser.de/ProductDetail/Micro-Commercial-Components-MCC/SK310A-TP?qs=O2qRfqcg9D9SKx4%252bV6P4XQ%3D%3D" H 2000 1300 50  0001 C CNN
+F 4 "SK310A-LTP" H 0   0   50  0001 C CNN "manf#"
 	1    2000 1300
 	1    0    0    -1
@@
 F 2 "heteromycin:SOT-669_LFPAK_ThermalVias-1" H 2400 1675 50  0001 L CIN
 F 3 "https://assets.nexperia.com/documents/data-sheet/PSMN1R2-30YLC.pdf" V 2200 1750 50  0001 L CNN
+F 4 "PSMN1R2-30YLC,115" H 0   0   50  0001 C CNN "manf#"
 	1    2200 1750
 	1    0    0    -1
@@
 F 2 "Resistor_SMD:R_0603_1608Metric" V 1430 1750 50  0001 C CNN
 F 3 "~" H 1500 1750 50  0001 C CNN
+F 4 "RC0603FR-7W100RL" H 0   0   50  0001 C CNN "manf#"
 	1    1500 1750
 	0    1    1    0
@@
 F 2 "Diode_SMD:D_SMA" H 2000 2950 50  0001 C CNN
 F 3 "https://www.mouser.de/ProductDetail/Micro-Commercial-Components-MCC/SK310A-TP?qs=O2qRfqcg9D9SKx4%252bV6P4XQ%3D%3D" H 2000 2950 50  0001 C CNN
+F 4 "SK310A-LTP" H 0   0   50  0001 C CNN "manf#"
 	1    2000 2950
 	1    0    0    -1
@@
 F 2 "Resistor_SMD:R_0603_1608Metric" V 1430 3400 50  0001 C CNN
 F 3 "~" H 1500 3400 50  0001 C CNN
+F 4 "RC0603FR-7W100RL" H 0   0   50  0001 C CNN "manf#"
 	1    1500 3400
 	0    1    1    0
@@
 F 2 "Resistor_SMD:R_0603_1608Metric" V 5080 1750 50  0001 C CNN
 F 3 "~" H 5150 1750 50  0001 C CNN
+F 4 "RC0603FR-7W100RL" H 0   0   50  0001 C CNN "manf#"
 	1    5150 1750
 	0    1    1    0
@@
 F 2 "Resistor_SMD:R_0603_1608Metric" V 5130 3400 50  0001 C CNN
 F 3 "~" H 5200 3400 50  0001 C CNN
+F 4 "RC0603FR-7W100RL" H 0   0   50  0001 C CNN "manf#"
 	1    5200 3400
 	0    1    1    0
@@
 F 2 "Resistor_SMD:R_0603_1608Metric" V 1880 2200 50  0001 C CNN
 F 3 "~" H 1950 2200 50  0001 C CNN
+F 4 "CRCW0603100KFKEAC" H 0   0   50  0001 C CNN "manf#"
 	1    1950 2200
 	0    1    1    0
@@
 F 2 "Resistor_SMD:R_0603_1608Metric" V 1880 3850 50  0001 C CNN
 F 3 "~" H 1950 3850 50  0001 C CNN
+F 4 "CRCW0603100KFKEAC" H 0   0   50  0001 C CNN "manf#"
 	1    1950 3850
 	0    1    1    0
@@
 F 2 "Resistor_SMD:R_0603_1608Metric" V 5530 2200 50  0001 C CNN
 F 3 "~" H 5600 2200 50  0001 C CNN
+F 4 "CRCW0603100KFKEAC" H 0   0   50  0001 C CNN "manf#"
 	1    5600 2200
 	0    1    1    0
@@
 F 2 "Resistor_SMD:R_0603_1608Metric" V 5580 3850 50  0001 C CNN
 F 3 "~" H 5650 3850 50  0001 C CNN
+F 4 "CRCW0603100KFKEAC" H 0   0   50  0001 C CNN "manf#"
 	1    5650 3850
 	0    1    1    0
@@
 F 2 "heteromycin:SOT-669_LFPAK_ThermalVias-1" H 2400 3325 50  0001 L CIN
 F 3 "https://assets.nexperia.com/documents/data-sheet/PSMN1R2-30YLC.pdf" V 2200 3400 50  0001 L CNN
+F 4 "PSMN1R2-30YLC,115" H 0   0   50  0001 C CNN "manf#"
 	1    2200 3400
 	1    0    0    -1
@@
 F 2 "Diode_SMD:D_SOD-123" H 5550 1300 50  0001 C CNN
 F 3 "https://www.mouser.de/datasheet/2/916/BAT54GW-1318921.pdf" H 5550 1300 50  0001 C CNN
+F 4 "BAT54GWJ" H 0   0   50  0001 C CNN "manf#"
 	1    5550 1300
 	1    0    0    -1
@@
 F 2 "Diode_SMD:D_SOD-123" H 5550 2950 50  0001 C CNN
 F 3 "https://www.mouser.de/datasheet/2/916/BAT54GW-1318921.pdf" H 5550 2950 50  0001 C CNN
+F 4 "BAT54GWJ" H 0   0   50  0001 C CNN "manf#"
 	1    5550 2950
 	1    0    0    -1
@@
 F 2 "Diode_SMD:D_SMA" H 2000 4450 50  0001 C CNN
 F 3 "https://www.mouser.de/ProductDetail/Micro-Commercial-Components-MCC/SK310A-TP?qs=O2qRfqcg9D9SKx4%252bV6P4XQ%3D%3D" H 2000 4450 50  0001 C CNN
+F 4 "SK310A-LTP" H 0   0   50  0001 C CNN "manf#"
 	1    2000 4450
 	1    0    0    -1
@@
 F 2 "Resistor_SMD:R_0603_1608Metric" V 1430 4900 50  0001 C CNN
 F 3 "~" H 1500 4900 50  0001 C CNN
+F 4 "RC0603FR-7W100RL" H 0   0   50  0001 C CNN "manf#"
 	1    1500 4900
 	0    1    1    0
@@
 F 2 "Resistor_SMD:R_0603_1608Metric" V 1880 5350 50  0001 C CNN
 F 3 "~" H 1950 5350 50  0001 C CNN
+F 4 "CRCW0603100KFKEAC" H 0   0   50  0001 C CNN "manf#"
 	1    1950 5350
 	0    1    1    0
@@
 F 2 "heteromycin:SOT-669_LFPAK_ThermalVias-1" H 2400 4825 50  0001 L CIN
 F 3 "https://assets.nexperia.com/documents/data-sheet/PSMN1R2-30YLC.pdf" V 2200 4900 50  0001 L CNN
+F 4 "PSMN1R2-30YLC,115" H 0   0   50  0001 C CNN "manf#"
 	1    2200 4900
 	1    0    0    -1
@@
 F 2 "Resistor_SMD:R_0603_1608Metric" V 7530 1750 50  0001 C CNN
 F 3 "~" H 7600 1750 50  0001 C CNN
+F 4 "RC0603FR-7W100RL" H 0   0   50  0001 C CNN "manf#"
 	1    7600 1750
 	0    1    1    0
@@
 F 2 "Resistor_SMD:R_0603_1608Metric" V 7580 3400 50  0001 C CNN
 F 3 "~" H 7650 3400 50  0001 C CNN
+F 4 "RC0603FR-7W100RL" H 0   0   50  0001 C CNN "manf#"
 	1    7650 3400
 	0    1    1    0
@@
 F 2 "Resistor_SMD:R_0603_1608Metric" V 7980 2200 50  0001 C CNN
 F 3 "~" H 8050 2200 50  0001 C CNN
+F 4 "CRCW0603100KFKEAC" H 0   0   50  0001 C CNN "manf#"
 	1    8050 2200
 	0    1    1    0
@@
 F 2 "Resistor_SMD:R_0603_1608Metric" V 8030 3850 50  0001 C CNN
 F 3 "~" H 8100 3850 50  0001 C CNN
+F 4 "CRCW0603100KFKEAC" H 0   0   50  0001 C CNN "manf#"
 	1    8100 3850
 	0    1    1    0
@@
 F 2 "Diode_SMD:D_SOD-123" H 8000 1300 50  0001 C CNN
 F 3 "https://www.mouser.de/datasheet/2/916/BAT54GW-1318921.pdf" H 8000 1300 50  0001 C CNN
+F 4 "BAT54GWJ" H 0   0   50  0001 C CNN "manf#"
 	1    8000 1300
 	1    0    0    -1
@@
 F 2 "Diode_SMD:D_SOD-123" H 8000 2950 50  0001 C CNN
 F 3 "https://www.mouser.de/datasheet/2/916/BAT54GW-1318921.pdf" H 8000 2950 50  0001 C CNN
+F 4 "BAT54GWJ" H 0   0   50  0001 C CNN "manf#"
 	1    8000 2950
 	1    0    0    -1
@@
 F 2 "Package_TO_SOT_SMD:SOT-23" H 5950 1850 50  0001 C CNN
 F 3 "https://www.infineon.com/dgdl/irlml0030pbf.pdf?fileId=5546d462533600a401535664773825df" H 5750 1750 50  0001 C CNN
+F 4 "IRLML0030TRPbF" H 0   0   50  0001 C CNN "manf#"
 	1    5750 1750
 	1    0    0    -1
@@
 F 2 "Package_TO_SOT_SMD:SOT-23" H 5950 3500 50  0001 C CNN
 F 3 "https://www.infineon.com/dgdl/irlml0030pbf.pdf?fileId=5546d462533600a401535664773825df" H 5750 3400 50  0001 C CNN
+F 4 "IRLML0030TRPbF" H 0   0   50  0001 C CNN "manf#"
 	1    5750 3400
 	1    0    0    -1
@@
 F 2 "Package_TO_SOT_SMD:SOT-23" H 8400 1850 50  0001 C CNN
 F 3 "https://www.infineon.com/dgdl/irlml0030pbf.pdf?fileId=5546d462533600a401535664773825df" H 8200 1750 50  0001 C CNN
+F 4 "IRLML0030TRPbF" H 0   0   50  0001 C CNN "manf#"
 	1    8200 1750
 	1    0    0    -1
@@
 F 2 "Package_TO_SOT_SMD:SOT-23" H 8400 3500 50  0001 C CNN
 F 3 "https://www.infineon.com/dgdl/irlml0030pbf.pdf?fileId=5546d462533600a401535664773825df" H 8200 3400 50  0001 C CNN
+F 4 "IRLML0030TRPbF" H 0   0   50  0001 C CNN "manf#"
 	1    8200 3400
 	1    0    0    -1
