File: power.sch (KiCad schematic (older format))
At the start: 33 parts, among them J2 4DB-P108-06, J3 39531-1002, J4 39531-1002, J5 Conn_02x03_Counter_Clockwise, U2 i3A, U3 AP7365-33WG-7

Commit message: Added manufacturer number to schematic
Parts:
- C10, C11, C3, C8, C9: manf# (none) -> VJ1812Y104KXBAT
- C12, C14: manf# (none) -> LMK316ABJ226KL-T
- C13: manf# (none) -> VJ1206Y104JXQCW1BC
- C15: manf# (none) -> EMK316BJ106MD-T
- C2, C4, C5, C6, C7: manf# (none) -> 860020573008
- D1, D2, D3: manf# (none) -> SMAJ28A-13-F
- D4: manf# (none) -> S3A-13-F
- D5: manf# (none) -> LTST-C194KGKT
- F1, F2, F3, F4: manf# (none) -> 3557-2
- FB1: manf# (none) -> MPZ1608S221A
- J2: manf# (none) -> 4DB-P108-06
- J3, J4: manf# (none) -> 039531-1002
- J5: manf# (none) -> 68602-406HLF
- R6: manf# (none) -> RC0603FR-1020KL
- R7: manf# (none) -> RC0603FR-0715KL
- R8: manf# (none) -> RC0603JR-7W1KL
- U2: manf# (none) -> I3A4W008A033V-001-R
- U3: manf# (none) -> AP7365-33WG-7
Changed lines of the file:
@@
 F 2 "Package_TO_SOT_SMD:SOT-23-5" H 7900 1850 50  0001 C CNN
 F 3 "https://www.mouser.de/datasheet/2/115/AP7365-86154.pdf" H 7900 1850 50  0001 C CNN
+F 4 "AP7365-33WG-7" H 0   0   50  0001 C CNN "manf#"
 	1    7900 1850
 	1    0    0    -1
@@
 F 2 "Capacitor_SMD:C_1206_3216Metric" H 4588 1250 50  0001 C CNN
 F 3 "~" H 4550 1400 50  0001 C CNN
+F 4 "LMK316ABJ226KL-T" H 0   0   50  0001 C CNN "manf#"
 	1    4550 1400
 	1    0    0    -1
@@
 F 2 "Capacitor_THT:CP_Radial_D6.3mm_P2.50mm" H 1538 1250 50  0001 C CNN
 F 3 "" H 1500 1400 50  0001 C CNN
+F 4 "860020573008" H 0   0   50  0001 C CNN "manf#"
 	1    1500 1400
 	1    0    0    -1
@@
 F 2 "Resistor_SMD:R_0603_1608Metric" V 8830 1900 50  0001 C CNN
 F 3 "~" H 8900 1900 50  0001 C CNN
+F 4 "RC0603JR-7W1KL" H 0   0   50  0001 C CNN "manf#"
 	1    8900 1900
 	1    0    0    -1
@@
 F 2 "LED_SMD:LED_0603_1608Metric" H 8900 2200 50  0001 C CNN
 F 3 "~" H 8900 2200 50  0001 C CNN
+F 4 "LTST-C194KGKT" H 0   0   50  0001 C CNN "manf#"
 	1    8900 2200
 	0    -1   -1   0
@@
 F 3 "https://www.mouser.de/datasheet/2/418/NG_CD_2-1437667-4_N8-639207.pdf" H 1200 4000 50  0001 C CNN
 F 4 "Alternative: OSTYK42106030" H 1200 4000 50  0001 C CNN "Note"
+F 5 "4DB-P108-06" H 0   0   50  0001 C CNN "manf#"
 	1    1200 4000
 	-1   0    0    -1
@@
 F 2 "heteromycin:KEYSTONE-FUSE-3557-2" V 2530 4400 50  0001 C CNN
 F 3 "~" H 2600 4400 50  0001 C CNN
+F 4 "3557-2" H 0   0   50  0001 C CNN "manf#"
 	1    2600 4400
 	0    1    1    0
@@
 F 2 "heteromycin:KEYSTONE-FUSE-3557-2" V 2530 3800 50  0001 C CNN
 F 3 "~" H 2600 3800 50  0001 C CNN
+F 4 "3557-2" H 0   0   50  0001 C CNN "manf#"
 	1    2600 3800
 	0    1    1    0
@@
 F 2 "heteromycin:KEYSTONE-FUSE-3557-2" V 2530 5600 50  0001 C CNN
 F 3 "~" H 2600 5600 50  0001 C CNN
+F 4 "3557-2" H 0   0   50  0001 C CNN "manf#"
 	1    2600 5600
 	0    1    1    0
@@
 F 2 "heteromycin:39531-1002" H 1200 4700 50  0001 C CNN
 F 3 "~" H 1200 4700 50  0001 C CNN
+F 4 "039531-1002" H 0   0   50  0001 C CNN "manf#"
 	1    1200 4700
 	-1   0    0    -1
@@
 F 2 "heteromycin:39531-1002" H 1200 5200 50  0001 C CNN
 F 3 "~" H 1200 5200 50  0001 C CNN
+F 4 "039531-1002" H 0   0   50  0001 C CNN "manf#"
 	1    1200 5200
 	-1   0    0    -1
@@
 F 2 "Diode_SMD:D_SMA" H 2950 3950 50  0001 C CNN
 F 3 "https://www.mouser.de/datasheet/2/240/Littelfuse_TVS_Diode_SMAJ_Datasheet.pdf-540740.pdf" H 2950 3950 50  0001 C CNN
+F 4 "SMAJ28A-13-F" H 0   0   50  0001 C CNN "manf#"
 	1    2950 3950
 	0    1    1    0
@@
 F 2 "Diode_SMD:D_SMA" H 2950 4550 50  0001 C CNN
 F 3 "https://www.mouser.de/datasheet/2/240/Littelfuse_TVS_Diode_SMAJ_Datasheet.pdf-540740.pdf" H 2950 4550 50  0001 C CNN
+F 4 "SMAJ28A-13-F" H 0   0   50  0001 C CNN "manf#"
 	1    2950 4550
 	0    1    1    0
@@
 F 2 "Capacitor_SMD:C_1812_4532Metric" H 4088 5600 50  0001 C CNN
 F 3 "" H 4050 5750 50  0001 C CNN
+F 4 "VJ1812Y104KXBAT" H 0   0   50  0001 C CNN "manf#"
 	1    4050 5750
 	1    0    0    -1
@@
 F 2 "Diode_SMD:D_SMC" H 2950 5750 50  0001 C CNN
 F 3 "https://www.mouser.de/datasheet/2/115/ds16005-37880.pdf" H 2950 5750 50  0001 C CNN
+F 4 "S3A-13-F" H 0   0   50  0001 C CNN "manf#"
 	1    2950 5750
 	0    1    1    0
@@
 F 2 "Capacitor_SMD:C_1812_4532Metric" H 4088 4400 50  0001 C CNN
 F 3 "" H 4050 4550 50  0001 C CNN
+F 4 "VJ1812Y104KXBAT" H 0   0   50  0001 C CNN "manf#"
 	1    4050 4550
 	1    0    0    -1
@@
 F 2 "Capacitor_SMD:C_1812_4532Metric" H 4088 3800 50  0001 C CNN
 F 3 "" H 4050 3950 50  0001 C CNN
+F 4 "VJ1812Y104KXBAT" H 0   0   50  0001 C CNN "manf#"
 	1    4050 3950
 	1    0    0    -1
@@
 F 2 "heteromycin:KEYSTONE-FUSE-3557-2" V 2530 5000 50  0001 C CNN
 F 3 "~" H 2600 5000 50  0001 C CNN
+F 4 "3557-2" H 0   0   50  0001 C CNN "manf#"
 	1    2600 5000
 	0    1    1    0
@@
 F 2 "Diode_SMD:D_SMA" H 2950 5150 50  0001 C CNN
 F 3 "https://www.mouser.de/datasheet/2/240/Littelfuse_TVS_Diode_SMAJ_Datasheet.pdf-540740.pdf" H 2950 5150 50  0001 C CNN
+F 4 "SMAJ28A-13-F" H 0   0   50  0001 C CNN "manf#"
 	1    2950 5150
 	0    1    1    0
@@
 F 2 "Capacitor_SMD:C_1812_4532Metric" H 4088 5000 50  0001 C CNN
 F 3 "" H 4050 5150 50  0001 C CNN
+F 4 "VJ1812Y104KXBAT" H 0   0   50  0001 C CNN "manf#"
 	1    4050 5150
 	1    0    0    -1
@@
 F 2 "Capacitor_THT:CP_Radial_D6.3mm_P2.50mm" H 3588 5000 50  0001 C CNN
 F 3 "" H 3550 5150 50  0001 C CNN
+F 4 "860020573008" H 0   0   50  0001 C CNN "manf#"
 	1    3550 5150
 	1    0    0    -1
@@
 F 2 "Capacitor_THT:CP_Radial_D6.3mm_P2.50mm" H 3588 4400 50  0001 C CNN
 F 3 "" H 3550 4550 50  0001 C CNN
+F 4 "860020573008" H 0   0   50  0001 C CNN "manf#"
 	1    3550 4550
 	1    0    0    -1
@@
 F 2 "Capacitor_THT:CP_Radial_D6.3mm_P2.50mm" H 3588 3800 50  0001 C CNN
 F 3 "" H 3550 3950 50  0001 C CNN
+F 4 "860020573008" H 0   0   50  0001 C CNN "manf#"
 	1    3550 3950
 	1    0    0    -1
@@
 F 2 "Capacitor_THT:CP_Radial_D6.3mm_P2.50mm" H 3588 5600 50  0001 C CNN
 F 3 "" H 3550 5750 50  0001 C CNN
+F 4 "860020573008" H 0   0   50  0001 C CNN "manf#"
 	1    3550 5750
 	1    0    0    -1
@@
 F 2 "Capacitor_SMD:C_1206_3216Metric" H 7038 1750 50  0001 C CNN
 F 3 "~" H 7000 1900 50  0001 C CNN
+F 4 "LMK316ABJ226KL-T" H 0   0   50  0001 C CNN "manf#"
 	1    7000 1900
 	1    0    0    -1
@@
 F 2 "Resistor_SMD:R_0603_1608Metric" V 6630 1750 50  0001 C CNN
 F 3 "https://www.mouser.de/datasheet/2/400/eads_commercial_power_mpz1608_en-923650.pdf" H 6700 1750 50  0001 C CNN
+F 4 "MPZ1608S221A" H 0   0   50  0001 C CNN "manf#"
 	1    6700 1750
 	0    1    1    0
@@
 F 2 "Capacitor_SMD:C_1206_3216Metric" H 8488 1750 50  0001 C CNN
 F 3 "~" H 8450 1900 50  0001 C CNN
+F 4 "EMK316BJ106MD-T " H 0   0   50  0001 C CNN "manf#"
 	1    8450 1900
 	1    0    0    -1
@@
 F 2 "Capacitor_SMD:C_1206_3216Metric" H 4988 1250 50  0001 C CNN
 F 3 "~" H 4950 1400 50  0001 C CNN
+F 4 "VJ1206Y104JXQCW1BC" H 0   0   50  0001 C CNN "manf#"
 	1    4950 1400
 	1    0    0    -1
@@
 F 2 "heteromycin:i3A" H 3000 1650 50  0001 C CNN
 F 3 "https://www.us.tdk-lambda.com/ftp/specs/i3a_full_datasheet.pdf" H 3000 1650 50  0001 C CNN
+F 4 "I3A4W008A033V-001-R" H 0   0   50  0001 C CNN "manf#"
 	1    3000 1650
 	1    0    0    -1
@@
 F 2 "Resistor_SMD:R_0603_1608Metric" V 3830 2000 50  0001 C CNN
 F 3 "~" H 3900 2000 50  0001 C CNN
+F 4 "RC0603FR-1020KL" H 0   0   50  0001 C CNN "manf#"
 	1    3900 2000
 	1    0    0    -1
@@
 F 2 "Resistor_SMD:R_0603_1608Metric" V 4080 2000 50  0001 C CNN
 F 3 "~" H 4150 2000 50  0001 C CNN
+F 4 "RC0603FR-0715KL" H 0   0   50  0001 C CNN "manf#"
 	1    4150 2000
 	1    0    0    -1
@@
 F 2 "Capacitor_SMD:C_1812_4532Metric" H 2088 1250 50  0001 C CNN
 F 3 "" H 2050 1400 50  0001 C CNN
+F 4 "VJ1812Y104KXBAT" H 0   0   50  0001 C CNN "manf#"
 	1    2050 1400
 	1    0    0    -1
@@
 F 2 "Connector_PinHeader_2.54mm:PinHeader_2x03_P2.54mm_Vertical" H 7750 3750 50  0001 C CNN
 F 3 "~" H 7750 3750 50  0001 C CNN
+F 4 "68602-406HLF" H 0   0   50  0001 C CNN "manf#"
 	1    7750 3750
 	1    0    0    -1
