File: sdcard.sch (KiCad schematic (older format))
At the start: 8 parts, among them J11 DM3D-SF

Commit message: Added manufacturer number to schematic
Parts:
- C111: manf# (none) -> EMK316BJ106MD-T
- J11: manf# (none) -> DM3D-SF
- R113, R114, R115, R116, R117, R118: manf# (none) -> CR0603-FX-4702ELF
Changed lines of the file:
@@
 F 2 "Connector_Card:microSD_HC_Hirose_DM3D-SF" H 8050 3850 50  0001 C CNN
 F 3 "https://www.hirose.com/product/en/download_file/key_name/DM3/category/Catalog/doc_file_id/49662/?file_category_id=4&item_id=195&is_series=1" H 6000 3250 50  0001 C CNN
+F 4 "DM3D-SF" H 0   0   50  0001 C CNN "manf#"
 	1    6000 3150
 	1    0    0    -1
@@
 F 2 "Resistor_SMD:R_0603_1608Metric" V 4780 2500 50  0001 C CNN
 F 3 "~" H 4850 2500 50  0001 C CNN
+F 4 "CR0603-FX-4702ELF" H 0   0   50  0001 C CNN "manf#"
 	1    4850 2500
 	-1   0    0    1
@@
 F 2 "Resistor_SMD:R_0603_1608Metric" V 4480 2500 50  0001 C CNN
 F 3 "~" H 4550 2500 50  0001 C CNN
+F 4 "CR0603-FX-4702ELF" H 0   0   50  0001 C CNN "manf#"
 	1    4550 2500
 	-1   0    0    1
@@
 F 2 "Resistor_SMD:R_0603_1608Metric" V 4180 2500 50  0001 C CNN
 F 3 "~" H 4250 2500 50  0001 C CNN
+F 4 "CR0603-FX-4702ELF" H 0   0   50  0001 C CNN "manf#"
 	1    4250 2500
 	-1   0    0    1
@@
 F 2 "Resistor_SMD:R_0603_1608Metric" V 3880 2500 50  0001 C CNN
 F 3 "~" H 3950 2500 50  0001 C CNN
+F 4 "CR0603-FX-4702ELF" H 0   0   50  0001 C CNN "manf#"
 	1    3950 2500
 	-1   0    0    1
@@
 F 2 "Resistor_SMD:R_0603_1608Metric" V 3580 2500 50  0001 C CNN
 F 3 "~" H 3650 2500 50  0001 C CNN
+F 4 "CR0603-FX-4702ELF" H 0   0   50  0001 C CNN "manf#"
 	1    3650 2500
 	-1   0    0    1
@@
 F 2 "Capacitor_SMD:C_1206_3216Metric" H 4438 3700 50  0001 C CNN
 F 3 "~" H 4400 3850 50  0001 C CNN
+F 4 "EMK316BJ106MD-T " H 0   0   50  0001 C CNN "manf#"
 	1    4400 3850
 	1    0    0    -1
@@
 F 2 "Resistor_SMD:R_0603_1608Metric" V 3280 2500 50  0001 C CNN
 F 3 "~" H 3350 2500 50  0001 C CNN
+F 4 "CR0603-FX-4702ELF" H 0   0   50  0001 C CNN "manf#"
 	1    3350 2500
 	-1   0    0    1
